Commit message: Added new updates to contingency planning, delta robots, franka interface, and frankapy.

File: manipulation/contingency_planning/assets/baseline_same_friction/block0.urdf (robot description, URDF)
Before this commit: robot block, 3 links, 2 joints
Links:
- link block1: mass 0.39196309669720986 -> 0.4593718160857386; geometry collision box size=0.14843942994035422 0.05 0.05; visual box size=0.14843942994035422 0.05 0.05
- link block2: mass 0.39196309669720986 -> 0.4593718160857386; geometry collision box size=0.0007802850298228914 0.05 0.05; visual box size=0.0007802850298228914 0.05 0.05
- link block3: mass 0.39196309669720986 -> 0.4593718160857386; geometry collision box size=0.0007802850298228914 0.05 0.05; visual box size=0.0007802850298228914 0.05 0.05
Joints:
- joint block_link1: origin xyz=0.04299431087457056 0.0 0.0 -> xyz=0.07460985748508855 0.0 0.0
- joint block_link2: origin xyz=0.06401137825085887 0.0 0.0 -> xyz=0.0007802850298228914 0.0 0.0

File: manipulation/contingency_planning/assets/baseline_same_friction/block1.urdf (robot description, URDF)
Before this commit: robot block, 3 links, 2 joints
Links:
- link block1: mass 2.0734609330105473 -> 0.8701614347119019; geometry collision box size=0.07361176209226883 0.05 0.05; visual box size=0.07361176209226883 0.05 0.05
- link block2: mass 0.3096664060786519 -> 0.8701614347119019; geometry collision box size=0.002776475815462337 0.05 0.05; visual box size=0.002776475815462337 0.05 0.05
- link block3: mass 0.3096664060786519 -> 1.0442516954117615; geometry collision box size=0.07361176209226883 0.05 0.05; visual box size=0.07361176209226883 0.05 0.05
Joints:
- joint block_link1: origin xyz=0.026621302232756678 0.0 0.0 -> xyz=0.03819411895386558 0.0 0.0
- joint block_link2: origin xyz=0.06168934888362166 0.0 0.0 -> xyz=0.03819411895386558 0.0 0.0

File: manipulation/contingency_planning/assets/baseline_same_friction/block10.urdf (robot description, URDF)
Before this commit: robot block, 3 links, 2 joints
Links:
- link block1: mass 0.4020555264806587 -> 0.8249515170605366; geometry collision box size=0.06276646309931407 0.05 0.05; visual box size=0.06276646309931407 0.05 0.05
- link block2: mass 0.4020555264806587 -> 0.8249515170605366; geometry collision box size=0.043616768450342965 0.05 0.05; visual box size=0.043616768450342965 0.05 0.05
- link block3: mass 0.4020555264806587 -> 0.16170825646809298; geometry collision box size=0.043616768450342965 0.05 0.05; visual box size=0.043616768450342965 0.05 0.05
Joints:
- joint block_link1: origin xyz=0.05213213616060974 0.0 0.0 -> xyz=0.05319161577482852 0.0 0.0
- joint block_link2: origin xyz=0.0457357276787805 0.0 0.0 -> xyz=0.043616768450342965 0.0 0.0

File: manipulation/contingency_planning/assets/baseline_same_friction/block11.urdf (robot description, URDF)
Before this commit: robot block, 3 links, 2 joints
Links:
- link block1: mass 1.1765680174696296 -> 0.9859235057217405; geometry collision box size=0.026478271353319083 0.05 0.05; visual box size=0.026478271353319083 0.05 0.05
- link block2: mass 0.30453870303707675 -> 0.9859235057217405; geometry collision box size=0.026478271353319083 0.05 0.05; visual box size=0.026478271353319083 0.05 0.05
- link block3: mass 0.30453870303707675 -> 0.9859235057217405; geometry collision box size=0.09704345729336183 0.05 0.05; visual box size=0.09704345729336183 0.05 0.05
Joints:
- joint block_link1: origin xyz=0.06526339643007069 0.0 0.0 -> xyz=0.026478271353319083 0.0 0.0
- joint block_link2: origin xyz=0.02458450487231848 0.0 0.0 -> xyz=0.06176086432334046 0.0 0.0

File: manipulation/contingency_planning/assets/baseline_same_friction/block12.urdf (robot description, URDF)
Before this commit: robot block, 3 links, 2 joints
Links:
- link block1: mass 0.5450482121348977 -> 0.665540940948494; geometry collision box size=0.04721877786417363 0.05 0.05; visual box size=0.04721877786417363 0.05 0.05
- link block2: mass 0.5450482121348977 -> 0.13046128750062572; geometry collision box size=0.04721877786417363 0.05 0.05; visual box size=0.04721877786417363 0.05 0.05
- link block3: mass 0.6476300486475821 -> 0.665540940948494; geometry collision box size=0.05556244427165273 0.05 0.05; visual box size=0.05556244427165273 0.05 0.05
Joints:
- joint block_link1: origin xyz=0.04276636826514474 0.0 0.0 -> xyz=0.04721877786417363 0.0 0.0
- joint block_link2: origin xyz=0.06446726346971052 0.0 0.0 -> xyz=0.05139061106791318 0.0 0.0

File: manipulation/contingency_planning/assets/baseline_same_friction/block13.urdf (robot description, URDF)
Before this commit: robot block, 3 links, 2 joints
Links:
- link block1: mass 2.2076574938802365 -> 1.0762063495042145; geometry collision box size=0.08598068125919699 0.05 0.05; visual box size=0.08598068125919699 0.05 0.05
- link block2: mass 0.5161081874698967 -> 0.5484950699613959; geometry collision box size=0.0372223181732801 0.05 0.05; visual box size=0.0372223181732801 0.05 0.05
- link block3: mass 0.23471340463179363 -> 0.5484950699613959; geometry collision box size=0.026797000567522905 0.05 0.05; visual box size=0.026797000567522905 0.05 0.05
Joints:
- joint block_link1: origin xyz=0.05882531589854447 0.0 0.0 -> xyz=0.061601499716238545 0.0 0.0
- joint block_link2: origin xyz=0.03234936820291105 0.0 0.0 -> xyz=0.032009659370401504 0.0 0.0

File: manipulation/contingency_planning/assets/baseline_same_friction/block14.urdf (robot description, URDF)
Before this commit: robot block, 3 links, 2 joints
Links:
- link block1: mass 0.9084268686753368 -> 0.8588296316353636; geometry collision box size=0.09898152618848019 0.05 0.05; visual box size=0.09898152618848019 0.05 0.05
- link block2: mass 0.9084268686753368 -> 0.5588497174172168; geometry collision box size=0.0255092369057599 0.05 0.05; visual box size=0.0255092369057599 0.05 0.05
- link block3: mass 0.9084268686753368 -> 0.5588497174172168; geometry collision box size=0.0255092369057599 0.05 0.05; visual box size=0.0255092369057599 0.05 0.05
Joints:
- joint block_link1: origin xyz=0.048226458030568436 0.0 0.0 -> xyz=0.062245381547120046 0.0 0.0
- joint block_link2: origin xyz=0.048226458030568436 0.0 0.0 -> xyz=0.0255092369057599 0.0 0.0

File: manipulation/contingency_planning/assets/baseline_same_friction/block15.urdf (robot description, URDF)
Before this commit: robot block, 3 links, 2 joints
Links:
- link block1: mass 0.6992965004437797 -> 0.21442710924437425; geometry collision box size=0.062834070009275 0.05 0.05; visual box size=0.062834070009275 0.05 0.05
- link block2: mass 0.6992965004437797 -> 0.21442710924437425; geometry collision box size=0.062834070009275 0.05 0.05; visual box size=0.062834070009275 0.05 0.05
- link block3: mass 1.099886871034901 -> 0.21442710924437425; geometry collision box size=0.024331859981449988 0.05 0.05; visual box size=0.024331859981449988 0.05 0.05
Joints:
- joint block_link1: origin xyz=0.07354052282493642 0.0 0.0 -> xyz=0.062834070009275 0.0 0.0
- joint block_link2: origin xyz=0.07354052282493642 0.0 0.0 -> xyz=0.043582964995362496 0.0 0.0

File: manipulation/contingency_planning/assets/baseline_same_friction/block16.urdf (robot description, URDF)
Before this commit: robot block, 3 links, 2 joints
Links:
- link block1: mass 0.5784772312537971 -> 0.7395218635635012; geometry collision box size=0.09826799081790921 0.05 0.05; visual box size=0.09826799081790921 0.05 0.05
- link block2: mass 0.8021748896769432 -> 0.7672021173586661; geometry collision box size=0.026726107660439775 0.05 0.05; visual box size=0.026726107660439775 0.05 0.05
- link block3: mass 0.8021748896769432 -> 0.7672021173586661; geometry collision box size=0.025005901521651008 0.05 0.05; visual box size=0.025005901521651008 0.05 0.05
Joints:
- joint block_link1: origin xyz=0.05276985763639576 0.0 0.0 -> xyz=0.06249704923917449 0.0 0.0
- joint block_link2: origin xyz=0.034096340157837246 0.0 0.0 -> xyz=0.02586600459104539 0.0 0.0

File: manipulation/contingency_planning/assets/baseline_same_friction/block17.urdf (robot description, URDF)
Before this commit: robot block, 3 links, 2 joints
Links:
- link block1: mass 0.987260073472935 -> 0.500920576326059; geometry collision box size=0.029244259788494084 0.05 0.05; visual box size=0.029244259788494084 0.05 0.05
- link block2: mass 1.3042722099810502 -> 0.44516159582267023; geometry collision box size=0.030540340307570336 0.05 0.05; visual box size=0.030540340307570336 0.05 0.05
- link block3: mass 0.10344489903128191 -> 0.500920576326059; geometry collision box size=0.09021539990393557 0.05 0.05; visual box size=0.09021539990393557 0.05 0.05
Joints:
- joint block_link1: origin xyz=0.014028998213555308 0.0 0.0 -> xyz=0.02989230004803221 0.0 0.0
- joint block_link2: origin xyz=0.06896714246071602 0.0 0.0 -> xyz=0.06037787010575295 0.0 0.0

File: manipulation/contingency_planning/assets/baseline_same_friction/block18.urdf (robot description, URDF)
Before this commit: robot block, 3 links, 2 joints
Links:
- link block1: mass 0.10042212050975985 -> 1.2056349207969195; geometry collision box size=0.0315855818355071 0.05 0.05; visual box size=0.0315855818355071 0.05 0.05
- link block2: mass 1.1495574836077624 -> 0.6836433542779207; geometry collision box size=0.0315855818355071 0.05 0.05; visual box size=0.0315855818355071 0.05 0.05
- link block3: mass 0.10042212050975985 -> 0.6836433542779207; geometry collision box size=0.08682883632898579 0.05 0.05; visual box size=0.08682883632898579 0.05 0.05
Joints:
- joint block_link1: origin xyz=0.06644007657335795 0.0 0.0 -> xyz=0.0315855818355071 0.0 0.0
- joint block_link2: origin xyz=0.06644007657335795 0.0 0.0 -> xyz=0.05920720908224644 0.0 0.0

File: manipulation/contingency_planning/assets/baseline_same_friction/block19.urdf (robot description, URDF)
Before this commit: robot block, 3 links, 2 joints
Links:
- link block1: mass 0.06895708343605234 -> 1.02410629585415; geometry collision box size=0.07055367558461768 0.05 0.05; visual box size=0.07055367558461768 0.05 0.05
- link block2: mass 0.06895708343605234 -> 0.7319479412644904; geometry collision box size=0.008892648830764627 0.05 0.05; visual box size=0.008892648830764627 0.05 0.05
- link block3: mass 2.827350095460671 -> 0.7319479412644904; geometry collision box size=0.07055367558461768 0.05 0.05; visual box size=0.07055367558461768 0.05 0.05
Joints:
- joint block_link1: origin xyz=0.046950405393004394 0.0 0.0 -> xyz=0.039723162207691155 0.0 0.0
- joint block_link2: origin xyz=0.0560991892139912 0.0 0.0 -> xyz=0.039723162207691155 0.0 0.0

File: manipulation/contingency_planning/assets/baseline_same_friction/block2.urdf (robot description, URDF)
Before this commit: robot block, 3 links, 2 joints
Links:
- link block1: mass 0.9035941964923446 -> 2.9998615020170862; geometry collision box size=0.12266028292154965 0.05 0.05; visual box size=0.12266028292154965 0.05 0.05
- link block2: mass 0.9035941964923446 -> 9.619892594909919e-05; geometry collision box size=0.013669858539225173 0.05 0.05; visual box size=0.013669858539225173 0.05 0.05
- link block3: mass 0.9035941964923446 -> 2.165333589334306e-05; geometry collision box size=0.013669858539225173 0.05 0.05; visual box size=0.013669858539225173 0.05 0.05
Joints:
- joint block_link1: origin xyz=0.010729257226393105 0.0 0.0 -> xyz=0.06816507073038741 0.0 0.0
- joint block_link2: origin xyz=0.06963537138680345 0.0 0.0 -> xyz=0.013669858539225173 0.0 0.0

File: manipulation/contingency_planning/assets/baseline_same_friction/block20.urdf (robot description, URDF)
Before this commit: robot block, 3 links, 2 joints
Links:
- link block1: mass 0.8155493049332374 -> 0.9385892410544447; geometry collision box size=0.03266657371859277 0.05 0.05; visual box size=0.03266657371859277 0.05 0.05
- link block2: mass 0.03379833149003728 -> 0.9385892410544447; geometry collision box size=0.08466685256281445 0.05 0.05; visual box size=0.08466685256281445 0.05 0.05
- link block3: mass 0.8155493049332374 -> 0.9385892410544447; geometry collision box size=0.03266657371859277 0.05 0.05; visual box size=0.03266657371859277 0.05 0.05
Joints:
- joint block_link1: origin xyz=0.06772838334481965 0.0 0.0 -> xyz=0.05866671314070361 0.0 0.0
- joint block_link2: origin xyz=0.06772838334481965 0.0 0.0 -> xyz=0.05866671314070361 0.0 0.0

File: manipulation/contingency_planning/assets/baseline_same_friction/block21.urdf (robot description, URDF)
Before this commit: robot block, 3 links, 2 joints
Links:
- link block1: mass 0.04389865767619734 -> 0.5171133875217969; geometry collision box size=0.026924460659066358 0.05 0.05; visual box size=0.026924460659066358 0.05 0.05
- link block2: mass 0.7858993794634778 -> 0.5171133875217969; geometry collision box size=0.09615107868186729 0.05 0.05; visual box size=0.09615107868186729 0.05 0.05
- link block3: mass 0.7858993794634778 -> 1.5948504979170925; geometry collision box size=0.026924460659066358 0.05 0.05; visual box size=0.026924460659066358 0.05 0.05
Joints:
- joint block_link1: origin xyz=0.07470752159561499 0.0 0.0 -> xyz=0.06153776967046682 0.0 0.0
- joint block_link2: origin xyz=0.037646239202192504 0.0 0.0 -> xyz=0.06153776967046682 0.0 0.0

File: manipulation/contingency_planning/assets/baseline_same_friction/block22.urdf (robot description, URDF)
Before this commit: robot block, 3 links, 2 joints
Links:
- link block1: mass 0.5042671931077441 -> 2.8770555563357503; geometry collision box size=0.06308601096977243 0.05 0.05; visual box size=0.06308601096977243 0.05 0.05
- link block2: mass 0.7523842265215616 -> 0.010937498315926482; geometry collision box size=0.02382797806045514 0.05 0.05; visual box size=0.02382797806045514 0.05 0.05
- link block3: mass 0.5042671931077441 -> 0.10058915313746143; geometry collision box size=0.06308601096977243 0.05 0.05; visual box size=0.06308601096977243 0.05 0.05
Joints:
- joint block_link1: origin xyz=0.06883020058575236 0.0 0.0 -> xyz=0.043456994515113784 0.0 0.0
- joint block_link2: origin xyz=0.04058489970712382 0.0 0.0 -> xyz=0.043456994515113784 0.0 0.0

File: manipulation/contingency_planning/assets/baseline_same_friction/block23.urdf (robot description, URDF)
Before this commit: robot block, 3 links, 2 joints
Links:
- link block1: mass 0.8039172566602181 -> 0.2962699303872225; geometry collision box size=0.08596567710055426 0.05 0.05; visual box size=0.08596567710055426 0.05 0.05
- link block2: mass 0.8039172566602181 -> 0.2962699303872225; geometry collision box size=0.04988423392764536 0.05 0.05; visual box size=0.04988423392764536 0.05 0.05
- link block3: mass 0.8039172566602181 -> 2.1673657295489797; geometry collision box size=0.014150088971800368 0.05 0.05; visual box size=0.014150088971800368 0.05 0.05
Joints:
- joint block_link1: origin xyz=0.06952384368330312 0.0 0.0 -> xyz=0.06792495551409981 0.0 0.0
- joint block_link2: origin xyz=0.010952312633393729 0.0 0.0 -> xyz=0.032017161449722865 0.0 0.0

File: manipulation/contingency_planning/assets/baseline_same_friction/block24.urdf (robot description, URDF)
Before this commit: robot block, 3 links, 2 joints
Links:
- link block1: mass 0.014290090066218397 -> 0.9544696463879542; geometry collision box size=0.011315850319243231 0.05 0.05; visual box size=0.011315850319243231 0.05 0.05
- link block2: mass 0.014290090066218397 -> 0.8663400272485957; geometry collision box size=0.06934207484037838 0.05 0.05; visual box size=0.06934207484037838 0.05 0.05
- link block3: mass 0.014290090066218397 -> 0.8663400272485957; geometry collision box size=0.06934207484037838 0.05 0.05; visual box size=0.06934207484037838 0.05 0.05
Joints:
- joint block_link1: origin xyz=0.07121485416783513 0.0 0.0 -> xyz=0.040328962579810806 0.0 0.0
- joint block_link2: origin xyz=0.07121485416783513 0.0 0.0 -> xyz=0.06934207484037838 0.0 0.0

File: manipulation/contingency_planning/assets/baseline_same_friction/block25.urdf (robot description, URDF)
Before this commit: robot block, 3 links, 2 joints
Links:
- link block1: mass 0.17808583342646164 -> 0.14268771281243198; geometry collision box size=0.04096031733149363 0.05 0.05; visual box size=0.04096031733149363 0.05 0.05
- link block2: mass 0.5716390896758681 -> 0.14268771281243198; geometry collision box size=0.04096031733149363 0.05 0.05; visual box size=0.04096031733149363 0.05 0.05
- link block3: mass 0.5716390896758681 -> 1.428472690703753; geometry collision box size=0.06807936533701274 0.05 0.05; visual box size=0.06807936533701274 0.05 0.05
Joints:
- joint block_link1: origin xyz=0.05102411303694649 0.0 0.0 -> xyz=0.04096031733149363 0.0 0.0
- joint block_link2: origin xyz=0.047951773926107014 0.0 0.0 -> xyz=0.05451984133425318 0.0 0.0

File: manipulation/contingency_planning/assets/baseline_same_friction/block26.urdf (robot description, URDF)
Before this commit: robot block, 3 links, 2 joints
Links:
- link block1: mass 0.568652061590856 -> 2.326316721897761; geometry collision box size=0.016286642969398194 0.05 0.05; visual box size=0.016286642969398194 0.05 0.05
- link block2: mass 0.18784774742128238 -> 0.4522996137149453; geometry collision box size=0.11742671406120361 0.05 0.05; visual box size=0.11742671406120361 0.05 0.05
- link block3: mass 0.568652061590856 -> 0.14895447971645834; geometry collision box size=0.016286642969398194 0.05 0.05; visual box size=0.016286642969398194 0.05 0.05
Joints:
- joint block_link1: origin xyz=0.03766973672757201 0.0 0.0 -> xyz=0.0668566785153009 0.0 0.0
- joint block_link2: origin xyz=0.03766973672757201 0.0 0.0 -> xyz=0.0668566785153009 0.0 0.0
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